File: KiCad Projects/GPIO_PROTECTION_RR/GPIO_PROTECTION_RR.kicad_sch (KiCad schematic)
At the start: 9 parts

Commit message: Design process
Parts:
- removed R2, R4: 330, symbol Device:R
- added C1: 100pf, Capacitor_SMD:C_0805_2012Metric, symbol Device:C
- added D2: PESD3V3S1UL, Package_TO_SOT_SMD:SOT-323_SC-70, symbol Diode:PESD3V3S1UL
- added D4: D, symbol Device:D
- added JP1: SolderJumper_2_Open, symbol Jumper:SolderJumper_2_Open
- added R10, R6: 10k, symbol Device:R
- added R2, R4, R5, R7, R8: 330, RC0805FR-07330RL:RESC2012X60N, symbol RC0805FR-07330RL:RC0805FR-07330RL
- added V5: 5, symbol Simulation_SPICE:VDC
- added VDD2: 3.3, symbol Simulation_SPICE:VDC
- V2: value 0 -> 5
Connections:
- net GND: now also C1.2, D2.2 (A), R10.2, R2.1, R6.2, V5.2, VDD2.2
- net at V1.1: now also R2.2
- net at V3.1: now also R4.1; no longer R3.1
- net at D1.2 (A): now also R3.1, R4.2; no longer V2.1
- new net: D2.1 (K), R8.1
- new net: JP1.2 (B), R8.2
- new net: D4.2 (A), R6.1, R7.2
- new net: C1.1, JP1.1 (A)
- new net: R5.1, V5.1
- new net: D4.1 (K), VDD2.1
- new net: R7.1, V2.1
- new net: R10.1, R5.2
Other:
- note added: "ACTUAL CIRCUIT FOR SURGE AND OVER VOLTAGE"
- note added: "SIMULATION CIRCUIT FOR SURGE AND OVER VOLTAGE"
- moved on the sheet: D1, R1, R3, V1, V3, VDD1

Commit message: Working
Parts:
- C1: value 100pf -> 100nf
- R8: value 330 -> 150
Connections:
- net EXT IN/OUT: now reaches D2.1 (K), R8.1
- net ESP32_GPIO: now reaches JP1.2 (B), R8.2
Changed lines of the file:
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@@
+	)
+	(junction
+		(at 58.42 33.02)
+		(diameter 0)
+		(color 0 0 0 0)
 	)
 	(junction
@@
 	(wire
 		(pts
+			(xy 49.53 33.02) (xy 58.42 33.02)
+		)
+		(stroke
+			(width 0)
+			(type default)
+		)
+	)
+	(wire
+		(pts
 			(xy 238.76 77.47) (xy 245.11 77.47)
 		)
@@
 			(width 0)
 			(type default)
+		)
+	)
+	(hierarchical_label "EXT IN{slash}OUT"
+		(shape bidirectional)
+		(at 49.53 33.02 180)
+		(effects
+			(font
+				(size 1.27 1.27)
+			)
+			(justify right)
+		)
+	)
+	(hierarchical_label "ESP32_GPIO"
+		(shape bidirectional)
+		(at 85.09 33.02 0)
+		(effects
+			(font
+				(size 1.27 1.27)
+			)
+			(justify left)
 		)
 	)
@@
 			)
 		)
-		(property "Value" "330"
+		(property "Value" "150"
 			(at 69.85 29.21 0)
 			(effects
@@
 			)
 		)
-		(property "Value" "100pf"
+		(property "Value" "100nf"
 			(at 85.09 48.2599 0)
 			(effects

Commit message: Working
Parts:
- removed R10: 10k, symbol Device:R
- removed R5: 330, RC0805FR-07330RL:RESC2012X60N, symbol RC0805FR-07330RL:RC0805FR-07330RL
- removed V5: 5, symbol Simulation_SPICE:VDC
- added D3: PESD3V3L2BT_215, PESD3V3L2BT:SOT95P230X110-3N, symbol PESD3V3L2BT_215:PESD3V3L2BT_215
Connections:
- net EXT IN/OUT: now also D3.3
- net GND: now also D3.2
- new net 3.3V: D3.1
- no-connect marks 0 -> 1
Other:
- moved on the sheet: C1, D2, JP1, R8
