File: KiCad Projects/FINAL_DESIGN/FINAL_DESIGN.kicad_pcb (KiCad board)
At the start: 2 copper layers, 123 parts, among them J1 Conn_01x19_Socket, J2 Conn_01x19_Socket, U1 ESP32_NODEMCU

Commit message: pcb design
Parts:
- added C31: 100nf, Capacitor_SMD:C_0805_2012Metric, F.Cu at (135.1, 167.0)
- added C32: 100nf, Capacitor_SMD:C_0805_2012Metric, F.Cu at (126.0, 166.5)
- added D31: D_Zener, Diode_SMD:D_SOD-882, F.Cu at (134.2, 154.0)
- added D32: D_Zener, Diode_SMD:D_SOD-882, F.Cu at (126.2, 154.5)
- added J3: Conn_01x19_Socket, Connector_PinHeader_2.54mm:PinHeader_1x19_P2.54mm_Vertical, F.Cu at (78.5, 60.2)
- added J4: Conn_01x19_Socket, Connector_PinHeader_2.54mm:PinHeader_1x19_P2.54mm_Vertical, F.Cu at (133.5, 60.9)
- added JP31: SolderJumper_2_Open, Jumper:SolderJumper-2_P1.3mm_Open_Pad1.0x1.5mm, F.Cu at (135.3, 162.0)
- added JP32: SolderJumper_2_Open, Jumper:SolderJumper-2_P1.3mm_Open_Pad1.0x1.5mm, F.Cu at (125.8, 162.0)
- added R31: 150, RC0805FR-07330RL:RESC2012X60N, F.Cu at (135.0, 157.5)
- added R32: 150, RC0805FR-07330RL:RESC2012X60N, F.Cu at (126.5, 157.5)
- moved U1 164.2 mm to (232.5, 60.5)
- moved JP9 129.3 mm to (73.0, 75.0)
- moved D26 127.3 mm to (235.7, 136.0)
- moved R9 127.2 mm to (72.7, 70.0)
- moved C9 126.5 mm to (72.7, 72.0)
- moved D25 119.0 mm to (227.2, 136.5)
- moved JP8 114.9 mm to (90.5, 63.0), turned to -90 degrees
- moved JP7 114.8 mm to (90.5, 59.6), turned to -90 degrees
- moved R8 112.9 mm to (87.5, 64.5)
- moved R7 112.7 mm to (87.5, 60.5)
- moved D24 112.2 mm to (220.2, 135.0)
- moved C8 111.7 mm to (87.5, 62.5), turned to 180 degrees
- moved C7 111.7 mm to (87.5, 58.5), turned to 180 degrees
- moved JP5 109.8 mm to (90.5, 76.5), turned to -90 degrees
- moved C6 108.5 mm to (86.5, 85.5), turned to 180 degrees
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- renumbered C36 to C10, C37 to C11, C38 to C12, C10 to C13, C2 to C14, C3 to C15, C4 to C16, C5 to C17, C6 to C18, C18 to C19, C7 to C2, C19 to C20, C20 to C21, C12 to C22, C13 to C23, C14 to C24, C15 to C25, C16 to C26, C11 to C27, C17 to C28, C25 to C29, C8 to C3, C26 to C30, C9 to C4, C31 to C5, C32 to C6, C33 to C7, C34 to C8, C35 to C9, D36 to D10, D37 to D11, D38 to D12, D10 to D13, D2 to D14, D3 to D15, D4 to D16, D5 to D17, D6 to D18, D18 to D19, D7 to D2, D19 to D20, D20 to D21, D12 to D22, D13 to D23, D14 to D24, D15 to D25, D16 to D26, D11 to D27, D17 to D28, D25 to D29, D8 to D3, D26 to D30, D9 to D4, D31 to D5, D32 to D6, D33 to D7, D34 to D8, D35 to D9, JP36 to JP10, JP37 to JP11, JP38 to JP12, JP10 to JP13, JP2 to JP14, JP3 to JP15, JP4 to JP16, JP5 to JP17, JP6 to JP18, JP18 to JP19, JP7 to JP2, JP19 to JP20, JP20 to JP21, JP12 to JP22, JP13 to JP23, JP14 to JP24, JP15 to JP25, JP16 to JP26, JP11 to JP27, JP17 to JP28, JP25 to JP29, JP8 to JP3, JP26 to JP30, JP9 to JP4, JP31 to JP5, JP32 to JP6, JP33 to JP7, JP34 to JP8, JP35 to JP9, R36 to R10, R37 to R11, R38 to R12, R10 to R13, R2 to R14, R3 to R15, R4 to R16, R5 to R17, R6 to R18, R18 to R19, R7 to R2, R19 to R20, R20 to R21, R12 to R22, R13 to R23, R14 to R24, R15 to R25, R16 to R26, R11 to R27, R17 to R28, R25 to R29, R8 to R3, R26 to R30, R9 to R4, R31 to R5, R32 to R6, R33 to R7, R34 to R8, R35 to R9
Connections:
- net /GPIO_EXTERN_0 renamed /I/O_0
- net /GPIO_EXTERN_1 renamed /TXD
- net /GPIO_EXTERN_10 renamed /SD3
- net /GPIO_EXTERN_11 renamed /CMD
- net /GPIO_EXTERN_12 renamed /I/O_12
- net /GPIO_EXTERN_13 renamed /I/O_13
- net /GPIO_EXTERN_14 renamed /I/O_14
- net /GPIO_EXTERN_15 renamed /I/O_15
- net /GPIO_EXTERN_16 renamed /I/O_16
- net /GPIO_EXTERN_17 renamed /I/O_17
- net /GPIO_EXTERN_18 renamed /I/O_18
- net /GPIO_EXTERN_19 renamed /I/O_19
- net /GPIO_EXTERN_2 renamed /I/O_2
- net /GPIO_EXTERN_21 renamed /I/O_21
- net /GPIO_EXTERN_22 renamed /I/O_22
- net /GPIO_EXTERN_23 renamed /I/O_23
- net /GPIO_EXTERN_25 renamed /I/O_25
- net /GPIO_EXTERN_26 renamed /I/O_26
- net /GPIO_EXTERN_27 renamed /I/O_27
- net /GPIO_EXTERN_3 renamed /RXD
- net /GPIO_EXTERN_32 renamed /I/O_32
- net /GPIO_EXTERN_33 renamed /I/O_33
- net /GPIO_EXTERN_34 renamed /I/O_34
- net /GPIO_EXTERN_35 renamed /I/O_35
- net /GPIO_EXTERN_4 renamed /I/O_4
- net /GPIO_EXTERN_5 renamed /I/O_5
- net /GPIO_EXTERN_6 renamed /CLK
- net /GPIO_EXTERN_7 renamed /SD0
- net /GPIO_EXTERN_8 renamed /SD1
- net /GPIO_EXTERN_9 renamed /SD2
- J2 pad 1: unconnected-(J2-Pin_1-Pad1) -> +3V3
Routing:
- net GND: track 0.00 -> 13.1 mm, vias 0 -> 12
- net /IO_9: track 0.00 -> 6.52 mm
- net /IO_2: track 0.00 -> 6.34 mm
- net /IO_3: track 0.00 -> 6.09 mm
- net /IO_4: track 0.00 -> 6.08 mm
- net /IO_7: track 0.00 -> 6.04 mm
- net /RXD: track 0.00 -> 5.88 mm
- net /IO_6: track 0.00 -> 5.82 mm
- net /IO_0: track 0.00 -> 5.78 mm
- net /IO_1: track 0.00 -> 5.78 mm
- net /TXD: track 0.00 -> 5.75 mm
- net Net-(JP10-A): track 0.00 -> 2.69 mm
- net Net-(JP3-A): track 0.00 -> 2.64 mm
- net Net-(JP1-A): track 0.00 -> 2.42 mm
- net Net-(JP4-A): track 0.00 -> 2.40 mm
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- added copper zone on B.Cu, net GND
Other:
- board outline added: 73.5 x 94.8 mm
- board text added: "ESP32_HEADERS"
- board text added: "EXTERNAL CONNECTOR1"
- board text added: "EXTERNAL CONNECTOR2"
