File: KiCad Projects/FINAL_DESIGN/FINAL_DESIGN.kicad_sch (KiCad schematic)
At the start: 123 parts, among them J1 Conn_01x19_Socket, J2 Conn_01x19_Socket, U1 ESP32_NODEMCU

Commit message: pcb design
Parts:
- added C31, C32: 100nf, Capacitor_SMD:C_0805_2012Metric, symbol Device:C
- added D31, D32: D_Zener, Diode_SMD:D_SOD-882, symbol Device:D_Zener
- added J3, J4: Conn_01x19_Socket, Connector_PinHeader_2.54mm:PinHeader_1x19_P2.54mm_Vertical, symbol Connector:Conn_01x19_Socket
- added JP31, JP32: SolderJumper_2_Open, Jumper:SolderJumper-2_P1.3mm_Open_Pad1.0x1.5mm, symbol Jumper:SolderJumper_2_Open
- added R31, R32: 150, RC0805FR-07330RL:RESC2012X60N, symbol RC0805FR-07330RL:RC0805FR-07330RL
- J1: footprint Connector_PinHeader_2.54mm:PinHeader_1x19_P2.54mm_Vertical -> Connector_PinSocket_2.54mm:PinSocket_1x19_P2.54mm_Vertical
- renumbered C36 to C10, C37 to C11, C38 to C12, C10 to C13, C2 to C14, C3 to C15, C4 to C16, C5 to C17, C6 to C18, C18 to C19, C7 to C2, C19 to C20, C20 to C21, C12 to C22, C13 to C23, C14 to C24, C15 to C25, C16 to C26, C11 to C27, C17 to C28, C25 to C29, C8 to C3, C26 to C30, C9 to C4, C31 to C5, C32 to C6, C33 to C7, C34 to C8, C35 to C9, D36 to D10, D37 to D11, D38 to D12, D10 to D13, D2 to D14, D3 to D15, D4 to D16, D5 to D17, D6 to D18, D18 to D19, D7 to D2, D19 to D20, D20 to D21, D12 to D22, D13 to D23, D14 to D24, D15 to D25, D16 to D26, D11 to D27, D17 to D28, D25 to D29, D8 to D3, D26 to D30, D9 to D4, D31 to D5, D32 to D6, D33 to D7, D34 to D8, D35 to D9, JP36 to JP10, JP37 to JP11, JP38 to JP12, JP10 to JP13, JP2 to JP14, JP3 to JP15, JP4 to JP16, JP5 to JP17, JP6 to JP18, JP18 to JP19, JP7 to JP2, JP19 to JP20, JP20 to JP21, JP12 to JP22, JP13 to JP23, JP14 to JP24, JP15 to JP25, JP16 to JP26, JP11 to JP27, JP17 to JP28, JP25 to JP29, JP8 to JP3, JP26 to JP30, JP9 to JP4, JP31 to JP5, JP32 to JP6, JP33 to JP7, JP34 to JP8, JP35 to JP9, R36 to R10, R37 to R11, R38 to R12, R10 to R13, R2 to R14, R3 to R15, R4 to R16, R5 to R17, R6 to R18, R18 to R19, R7 to R2, R19 to R20, R20 to R21, R12 to R22, R13 to R23, R14 to R24, R15 to R25, R16 to R26, R11 to R27, R17 to R28, R25 to R29, R8 to R3, R26 to R30, R9 to R4, R31 to R5, R32 to R6, R33 to R7, R34 to R8, R35 to R9
Connections:
- net EN: now also J4.2 (Pin_2)
- net GND: now also C31.2, C32.2, D31.2 (A), D32.2 (A), J3.13 (Pin_13), J3.19 (Pin_19), J4.14 (Pin_14)
- net IO_36: now also JP31.2 (B), R31.2
- net IO_39: now also JP32.2 (B), R32.2
- net VIN 5V: now also J4.19 (Pin_19)
- net +3V3: now reaches J2.1 (Pin_1)
- net +3V3: now also J4.1 (Pin_1)
- net GPIO_EXTERN_0 renamed I/O_0
- net I/O_0: now also J3.6 (Pin_6)
- net GPIO_EXTERN_1 renamed TXD
- net TXD: now also J3.16 (Pin_16)
- net GPIO_EXTERN_10 renamed SD3
- net SD3: now also J4.17 (Pin_17)
- net GPIO_EXTERN_11 renamed CMD
- net CMD: now also J4.18 (Pin_18)
- net GPIO_EXTERN_12 renamed I/O_12
- net I/O_12: now also J4.13 (Pin_13)
- net GPIO_EXTERN_13 renamed I/O_13
- net I/O_13: now also J4.15 (Pin_15)
- net GPIO_EXTERN_14 renamed I/O_14
- net I/O_14: now also J4.12 (Pin_12)
- net GPIO_EXTERN_15 renamed I/O_15
- net I/O_15: now also J3.4 (Pin_4)
- net GPIO_EXTERN_16 renamed I/O_16
- net I/O_16: now also J3.8 (Pin_8)
- net GPIO_EXTERN_17 renamed I/O_17
- net I/O_17: now also J3.9 (Pin_9)
- net GPIO_EXTERN_18 renamed I/O_18
- net I/O_18: now also J3.11 (Pin_11)
- net GPIO_EXTERN_19 renamed I/O_19
- net I/O_19: now also J3.12 (Pin_12)
- net GPIO_EXTERN_2 renamed I/O_2
- net I/O_2: now also J3.5 (Pin_5)
- net GPIO_EXTERN_21 renamed I/O_21
- net I/O_21: now also J3.14 (Pin_14)
- net GPIO_EXTERN_22 renamed I/O_22
- net I/O_22: now also J3.17 (Pin_17)
- net GPIO_EXTERN_23 renamed I/O_23
- net I/O_23: now also J3.18 (Pin_18)
- net GPIO_EXTERN_25 renamed I/O_25
- net I/O_25: now also J4.9 (Pin_9)
- net GPIO_EXTERN_26 renamed I/O_26
- net I/O_26: now also J4.10 (Pin_10)
- net GPIO_EXTERN_27 renamed I/O_27
- net I/O_27: now also J4.11 (Pin_11)
- net GPIO_EXTERN_3 renamed RXD
- net RXD: now also J3.15 (Pin_15)
- net GPIO_EXTERN_32 renamed I/O_32
- net I/O_32: now also J4.7 (Pin_7)
- net GPIO_EXTERN_33 renamed I/O_33
- net I/O_33: now also J4.8 (Pin_8)
- net GPIO_EXTERN_34 renamed I/O_34
- net I/O_34: now also J4.5 (Pin_5)
- net GPIO_EXTERN_35 renamed I/O_35
- net I/O_35: now also J4.6 (Pin_6)
- net GPIO_EXTERN_4 renamed I/O_4
- net I/O_4: now also J3.7 (Pin_7)
- net GPIO_EXTERN_5 renamed I/O_5
- net I/O_5: now also J3.10 (Pin_10)
- net GPIO_EXTERN_6 renamed CLK
- net CLK: now also J3.1 (Pin_1)
- net GPIO_EXTERN_7 renamed SD0
- net SD0: now also J3.2 (Pin_2)
- net GPIO_EXTERN_8 renamed SD1
- net SD1: now also J3.3 (Pin_3)
- net GPIO_EXTERN_9 renamed SD2
- net SD2: now also J4.16 (Pin_16)
- new net: C31.1, JP31.1 (A)
- new net: C32.1, JP32.1 (A)
- new net SN: D32.1 (K), J4.4 (Pin_4), R32.1
- new net SP: D31.1 (K), J4.3 (Pin_3), R31.1
Other:
- company: (none) -> KCT
- title: (none) -> ESP32 CARRIER BOARD
- moved on the sheet: C13, D13, JP13, R13
