File: KiCad Projects/FINAL_DESIGN/FINAL_DESIGN.kicad_sch (KiCad schematic)
At the start: 147 parts, among them J1 Screw_Terminal_01x02, J2 Conn_01x19_Socket, J3 Conn_01x19_Socket, J4 Conn_01x19_Socket, J5 Conn_01x19_Socket, Q1 PMOS, U1 DC_DC_small, U2 ESP32_NODEMCU

Commit message: Design
Parts:
- removed U1: DC_DC_small, DC_DC_LM2596_small:DC_DC_LM2596_small, symbol LM2596_Module:DC_DC_small
